File: PCB/ESP32 DSP Board/ESP32 DSP Board.kicad_sch (KiCad schematic)
At the start: 76 parts, among them J1 USB4216-03-A_REVA, J2 USB4216-03-A_REVA, SW1 PTS810_SJM_250_SMTR_LFS, SW2 PTS810_SJM_250_SMTR_LFS, U11 INTERFACE-CP2102-GMR_QFN28_, U8 ESP32-S3-WROOM-1, U9 TPS73733DCQ

Commit message: Schematic finished, footprints associated to components, PCB updated from schematic
Parts:
- removed C1, C10, C11, C2: 0.1uF, symbol Device:C
- removed R1, R2, R8, R9: 22/33, symbol Device:R
- removed R13: 1K, symbol Device:R
- C12, C15, C3, C4, C5, C6: footprint (none) -> Capacitor_SMD:C_0805_2012Metric
- C13, C14: value C -> 0.1uF; footprint (none) -> Capacitor_SMD:C_01005_0402Metric
- C16: value C -> 10uF; footprint (none) -> Capacitor_SMD:C_0805_2012Metric
- C17, C18, C19, C20, C21, C7, C9: footprint (none) -> Capacitor_SMD:C_01005_0402Metric
- D1, D2, D4: footprint (none) -> LED_SMD:LED_0805_2012Metric
- D3: footprint (none) -> LED_SMD:LED_0603_1608Metric
- J1, J2: footprint USB4216-03-A_REVA:GCT_USB4216-03-A_REVA -> USB_Connector:GCT_USB4216-03-A_REVA
- J3: footprint (none) -> Connector_PinHeader_2.54mm:PinHeader_1x04_P2.54mm_Vertical
- J4: footprint (none) -> Connector_PinSocket_2.54mm:PinSocket_1x02_P2.54mm_Vertical
- J5: footprint (none) -> Connector_PinHeader_2.54mm:PinHeader_1x02_P2.54mm_Vertical
- J6: footprint (none) -> Connector_PinHeader_2.54mm:PinHeader_1x16_P2.54mm_Vertical
- J7: footprint (none) -> Connector_PinSocket_2.54mm:PinSocket_1x04_P2.54mm_Vertical
- R10, R11, R15, R17, R18, R19, R24, R25, R26, R27, R29, R3, R30, R31, R4, R7: footprint (none) -> Resistor_SMD:R_0805_2012Metric
- R12, R14, R16, R28, R5, R6: footprint (none) -> Resistor_SMD:R_0603_1608Metric
- R20: value R -> 2K; footprint (none) -> Resistor_SMD:R_0805_2012Metric
- R21: value R -> 10K; footprint (none) -> Resistor_SMD:R_0805_2012Metric
- R22: value R -> 15K; footprint (none) -> Resistor_SMD:R_0805_2012Metric
- R23: value R -> 22K; footprint (none) -> Resistor_SMD:R_0805_2012Metric
- SW1, SW2: footprint PTS810_SJM_250_SMTR_LFS:SW_PTS810_SJM_250_SMTR_LFS -> Switches:SW_PTS810_SJM_250_SMTR_LFS
- U1: footprint (none) -> Package_DIP:CERDIP-16_W7.62mm_SideBrazed
- U10, U12: footprint (none) -> USB_ESD:USBLC6-2P6
- U11: footprint INTERFACE-CP2102-GMR_QFN28_:QFN28G_0.5-5X5MM -> USB-UART-Bridge:CP2102-QFN28G
- U2: footprint (none) -> Package_DIP:CERDIP-14_W7.62mm_SideBrazed
- U3: footprint (none) -> Package_DIP:CERDIP-8_W7.62mm_SideBrazed
- U4, U5, U7: footprint (none) -> Package_DIP:DIP-8_W7.62mm
- U6: footprint (none) -> Package_DIP:DIP-16_W7.62mm
- U9: footprint TPS73733DCQ:SOT127P706X180-6N -> LDO_3V3:TPS73733DCQ
Connections:
- net at J1.A7 (DN1), J1.B7 (DN2): now also U10.4 (I/O2)
- net at U12.3 (I/O2): now also J2.A6 (DP1), J2.B6 (DP2)
- net at U12.4 (I/O2): now also J2.A7 (DN1), J2.B7 (DN2)
- net at U10.3 (I/O2): now also J1.A6 (DP1), J1.B6 (DP2)

Commit message: Added clamping and biasing to audio inputs, hpf and rail to rail amplifier to DAC output, 1.5V LDO, footprints updated
Parts:
- removed J2: USB4216-03-A_REVA, USB_Connector:GCT_USB4216-03-A_REVA, symbol USB4216-03-A_REVA:USB4216-03-A_REVA
- removed J3: ~, Connector_PinHeader_2.54mm:PinHeader_1x04_P2.54mm_Vertical, symbol Terminal_Block_Generic:4-Way-Screw-Block
- removed J6: ~, Connector_PinHeader_2.54mm:PinHeader_1x16_P2.54mm_Vertical, symbol Pin_Header_Generic:16_Pin_Header
- removed U11: INTERFACE-CP2102-GMR_QFN28_, USB-UART-Bridge:CP2102-QFN28G, symbol INTERFACE-CP2102-GMR_QFN28_:INTERFACE-CP2102-GMR_QFN28_
- removed U12: ~, USB_ESD:USBLC6-2P6, symbol ESD_Protection_STM:USBLC-2
- removed U5: ~, Package_DIP:DIP-8_W7.62mm, symbol Amplifier_Operational_Renesas:CA3140A
- added C1, C11, C2: 10uF, Capacitor_SMD:C_0603_1608Metric, symbol Device:C
- added C10, C22, C23, C24, C25, C26, C27: 0.1uF, Capacitor_SMD:C_0402_1005Metric, symbol Device:C
- added C28: 10nF, Capacitor_SMD:C_0402_1005Metric, symbol Device:C
- added C8: 1uF, Capacitor_SMD:C_0603_1608Metric, symbol Device:C
- added D10, D5, D6, D7, D8, D9: D_Zener, Diode_SMD:D_SOD-123, symbol Device:D_Zener
- added J2: ~, Connector_PinHeader_2.54mm:PinHeader_1x18_P2.54mm_Vertical, symbol Pin_Header_Generic:18_pin_header
- added J3: ~, Connector_PinHeader_2.54mm:PinHeader_1x05_P2.54mm_Vertical, symbol Pin_Header_Generic:5_Pin_Header
- added R1, R13, R2, R8, R9: 10K, Resistor_SMD:R_0402_1005Metric, symbol Device:R
- added R32: 95.3K, Resistor_SMD:R_0402_1005Metric, symbol Device:R
- added U12: ~, Package_DIP:CERDIP-8_W7.62mm_SideBrazed, symbol Amplifier_Operational_TI:OPA705PA
- added U5: ~, LDO_Adjustable:TPS73601DBVT, symbol LDO_TI:TPS736
- C12: value 10uF -> 0.1uF; footprint Capacitor_SMD:C_0805_2012Metric -> Capacitor_SMD:C_0402_1005Metric
- C15, C16, C3, C4, C5: footprint Capacitor_SMD:C_0805_2012Metric -> Capacitor_SMD:C_0603_1608Metric
- R10, R11: value 5.1k -> 10K; footprint Resistor_SMD:R_0805_2012Metric -> Resistor_SMD:R_0402_1005Metric
- R12: value 1K -> 10K; footprint Resistor_SMD:R_0603_1608Metric -> Resistor_SMD:R_0402_1005Metric
- R14, R5, R6: footprint Resistor_SMD:R_0603_1608Metric -> Resistor_SMD:R_0402_1005Metric
- R15: value 470 -> 1K; footprint Resistor_SMD:R_0805_2012Metric -> Resistor_SMD:R_0402_1005Metric
- R16: value 220 -> 23.2K; footprint Resistor_SMD:R_0603_1608Metric -> Resistor_SMD:R_0402_1005Metric
- R17, R18, R19, R20, R21, R22, R23, R24, R25, R26, R27, R29, R3, R30, R31, R4, R7: footprint Resistor_SMD:R_0805_2012Metric -> Resistor_SMD:R_0402_1005Metric
- R28: footprint Resistor_SMD:R_0603_1608Metric -> Resistor_SMD:R_0805_2012Metric
Connections:
- net +3.3V: no longer R12.2
- net +3V3: no longer C12.1
- net +5V: now also C12.1, C10.2, C22.1, C23.1, C27.1, U5.1 (In), U5.3 (En); no longer R16.2
- net ADC CH0: now also J3.1
- net ADC CH1: now also J3.2
- net ADC CH2: now also J3.3
- net ADC CH3: now also J3.4
- net DAC OUT: now also U12.3 (In+); no longer J5.1
- net ESP Rx: now also J2.18
- net ESP Tx: now also J2.17
- net GND: now also R15.2, C10.1, C11.2, C22.2, C23.2, C24.2, C25.2, C26.2, C27.2, C28.2, D10.2 (A), D6.2 (A), D7.2 (A), D9.2 (A), J2.16, J3.5, R2.2, R32.2, U12.4 (V-), U5.2 (GND); no longer R10.1
- net IO10: now also J2.13
- net IO11: now also J2.14
- net IO12: now also J2.15
- net IO15: now also J2.5
- net IO16: now also J2.6
- net IO17: now also J2.7
- net IO18: now also J2.8
- net IO3: now also J2.10
- net IO4: now also J2.1
- net IO46: now also J2.11
- net IO5: now also J2.2
- net IO6: now also J2.3
- net IO7: now also J2.4
- net IO8: now also J2.9
- net IO9: now also J2.12
- net USB D-: now also U10.3 (I/O2); no longer U10.6 (I/O1)
- net VDD: now also C24.1, C25.1, C26.1, U12.7 (V+)
- net at R12.1: now also C2.2, R13.1
- net CH0_FOUT: now reaches C18.2, U4.1 (1OUT)
- net CH0_FOUT: now also U4.2 (1IN-), R1.1; no longer U2.1 (CH0)
- net CH1_FOUT: now reaches C20.2, U4.7 (2OUT)
- net CH1_FOUT: now also R10.1, U4.5 (2IN+); no longer U2.2 (CH1)
- net at R19.2, U6.3 (Y_OUT/IN): now also U12.2 (In-)
- net at R10.2: now also R11.1, C2.1, D8.2 (A)
- net at J1.A6 (DP1), J1.B6 (DP2): now also U10.6 (I/O1); no longer U10.3 (I/O2)
- net 1.5V: now reaches R16.1
- net 1.5V: now also R12.2, C11.1, C28.1, R8.2, U5.5 (Out); no longer R15.2
- net at R15.1: now also J5.1, C8.1; no longer U3.1 (Zener_Cathode)
- net CH0 OUT: no longer names the net of R20.1, R21.1, R22.1, R23.1
- net CH0 OUT: now also C8.2, U12.6 (OUT)
- new net: D5.1 (K), D6.1 (K)
- new net: R16.2, R32.1, U5.4 (NR/FB)
- new net: C1.1, D5.2 (A), R1.2, R2.1
- new net: C1.2, R8.1, R9.1
- new net: D8.1 (K), D9.1 (K)
- new net CH0 IN: D7.1 (K), R9.2, U2.1 (CH0)
- new net CH1 IN: D10.1 (K), R13.2, U2.2 (CH1)
Other:
- note removed: "USB-UART Bridge"
- moved on the sheet: C13, C14, C15, C16, C17, C18, C19, C20, C21, C3, C4, C5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

Commit message: pcb component layout finished, ic and pin header footprints fixed
Parts:
- J4: footprint Connector_PinSocket_2.54mm:PinSocket_1x02_P2.54mm_Vertical -> Connector_PinHeader_2.54mm:PinHeader_1x02_P2.54mm_Vertical
- J7: footprint Connector_PinSocket_2.54mm:PinSocket_1x04_P2.54mm_Vertical -> Connector_PinHeader_2.54mm:PinHeader_1x04_P2.54mm_Vertical
- U1: footprint Package_DIP:CERDIP-16_W7.62mm_SideBrazed -> Package_DIP:DIP-16_W7.62mm
- U12, U3: footprint Package_DIP:CERDIP-8_W7.62mm_SideBrazed -> Package_DIP:DIP-8_W7.62mm
- U2: footprint Package_DIP:CERDIP-14_W7.62mm_SideBrazed -> Package_DIP:DIP-14_W7.62mm
Changed lines of the file:
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@@
 			)
 		)
-		(property "Footprint" "Package_DIP:CERDIP-14_W7.62mm_SideBrazed"
+		(property "Footprint" "Package_DIP:DIP-14_W7.62mm"
 			(at 36.83 97.79 0)
 			(effects
@@
 			)
 		)
-		(property "Footprint" "Connector_PinSocket_2.54mm:PinSocket_1x02_P2.54mm_Vertical"
+		(property "Footprint" "Connector_PinHeader_2.54mm:PinHeader_1x02_P2.54mm_Vertical"
 			(at 270.51 264.16 0)
 			(effects
@@
 			)
 		)
-		(property "Footprint" "Connector_PinSocket_2.54mm:PinSocket_1x04_P2.54mm_Vertical"
+		(property "Footprint" "Connector_PinHeader_2.54mm:PinHeader_1x04_P2.54mm_Vertical"
 			(at 254 260.35 0)
 			(effects
@@
 			)
 		)
-		(property "Footprint" "Package_DIP:CERDIP-8_W7.62mm_SideBrazed"
+		(property "Footprint" "Package_DIP:DIP-8_W7.62mm"
 			(at 57.15 45.72 0)
 			(effects
@@
 			)
 		)
-		(property "Footprint" "Package_DIP:CERDIP-16_W7.62mm_SideBrazed"
+		(property "Footprint" "Package_DIP:DIP-16_W7.62mm"
 			(at 114.3 45.72 0)
 			(effects
@@
 			)
 		)
-		(property "Footprint" "Package_DIP:CERDIP-8_W7.62mm_SideBrazed"
+		(property "Footprint" "Package_DIP:DIP-8_W7.62mm"
 			(at 234.95 53.34 0)
 			(effects
