File: PCB/ESP32 DSP Board/ESP32 DSP Board.kicad_pcb (KiCad board)
At the start: 6 copper layers, 165.8 x 86 mm, 77 parts, among them U8 ESP32-S3-WROOM-1

Commit message: latest commit before laptop migration
Parts:
- added J1: USB4216-03-A_REVA, USB_Connector:GCT_USB4216-03-A_REVA, F.Cu at (153.8, 61.3)
- added SW1: PTS810_SJM_250_SMTR_LFS, Switches:SW_PTS810_SJM_250_SMTR_LFS, F.Cu at (161.1, 84.8)
- added SW2: PTS810_SJM_250_SMTR_LFS, Switches:SW_PTS810_SJM_250_SMTR_LFS, F.Cu at (154.1, 118.3)
- added U9: TPS73733DCQ, LDO_3V3:TPS73733DCQ, F.Cu at (153.1, 78.0)
- D1, D2, D4: footprint LED_SMD:LED_0805_2012Metric -> LED_SMD:LED_1206_3216Metric_Pad1.42x1.75mm_HandSolder
- D3: footprint LED_SMD:LED_0603_1608Metric -> LED_SMD:LED_1206_3216Metric_Pad1.42x1.75mm_HandSolder
- moved C20 296.9 mm to (92.9, 129.5), turned to 90 degrees
- moved C28 296.7 mm to (92.0, 109.8), turned to 180 degrees
- moved C26 292.5 mm to (94.8, 97.6)
- moved C21 292.1 mm to (99.1, 135.6)
- moved C29 291.7 mm to (97.5, 114.0), turned to 180 degrees
- moved C30 290.5 mm to (99.6, 119.9), turned to -90 degrees
- moved C23 287.1 mm to (99.0, 128.2), turned to 180 degrees
- moved C1 280.6 mm to (99.0, 124.2), turned to 180 degrees
- moved U7 279.9 mm to (83.3, 97.8)
- moved D4 279.9 mm to (72.5, 102.5), turned to 90 degrees
- moved J4 279.4 mm to (77.5, 87.2)
- moved C18 277.5 mm to (115.8, 127.5)
- moved J5 276.1 mm to (85.5, 77.8), turned to -90 degrees
- moved J3 274.4 mm to (113.0, 141.1), turned to -90 degrees
- moved C25 272.3 mm to (102.7, 94.4)
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Routing:
- net GND: track 0.00 -> 160.2 mm
- net ADC CH2: track 36.4 -> 0.00 mm
- net IO9: track 34.6 -> 0.00 mm
- net IO10: track 31.6 -> 0.00 mm
- net CH0_FOUT: track 0.00 -> 31.6 mm
- net Net-(U3-C-): track 0.00 -> 31.2 mm
- net ADC CH3: track 31.2 -> 0.00 mm
- net DB4: track 0.00 -> 29.2 mm
- net DB2: track 29.2 -> 0.00 mm
- net DB1: track 25.9 -> 0.00 mm
- net DB0: track 25.5 -> 0.00 mm
- net IO11: track 21.3 -> 0.00 mm
- net CH1_FOUT: track 0.00 -> 21.3 mm
- net IO35: track 19.2 -> 0.00 mm
- net DB3: track 18.6 -> 0.00 mm
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Other:
- board size 165.8 x 86 mm -> 120.7 x 86.6 mm
